File: pcb/Wireless232/Wireless232.sch (KiCad schematic (older format))
At the start: 16 parts, among them J1 Power, J2 DTE Connector, J3 DCE Connector, U1 ESP32_DevKitC, U2 MAX202

Commit message: PCB Tidy, improved examples for laser monitoring
Connections:
- net at U1.13 (IO12): no longer R3.2
- net ESP_TX: now reaches U1.17 (SD3/IO10/TXD1)
- net ESP_TX: now also R3.2
Other:
- moved on the sheet: R3
Changed lines of the file:
@@
 L Device:R R3
 U 1 1 5E6093E8
-P 4800 2950
-F 0 "R3" V 4850 3150 50  0000 C CNN
-F 1 "0R" V 4800 2950 50  0000 C CNN
-F 2 "Resistor_SMD:R_1206_3216Metric" V 4730 2950 50  0001 C CNN
-F 3 "~" H 4800 2950 50  0001 C CNN
-	1    4800 2950
+P 5400 2850
+F 0 "R3" V 5450 3050 50  0000 C CNN
+F 1 "0R" V 5400 2850 50  0000 C CNN
+F 2 "Resistor_SMD:R_1206_3216Metric" V 5330 2850 50  0001 C CNN
+F 3 "~" H 5400 2850 50  0001 C CNN
+	1    5400 2850
 	0    1    1    0
 $EndComp
@@
 Wire Wire Line
 	6100 3450 5650 3450
-Wire Wire Line
-	5650 3450 5650 2950
-Wire Wire Line
-	5650 2950 4950 2950
 Wire Wire Line
 	4950 3150 5400 3150
@@
 NoConn ~ 3000 4250
 NoConn ~ 3000 4350
-NoConn ~ 3000 4450
 NoConn ~ 3000 4550
 NoConn ~ 4650 4850
@@
 NoConn ~ 4650 3500
 NoConn ~ 4650 3400
+Wire Wire Line
+	5650 2850 5550 2850
+Wire Wire Line
+	5650 2850 5650 3450
+Text Label 4900 2850 0    50   ~ 0
+ESP_TX
+Wire Wire Line
+	4900 2850 5250 2850
+Text Label 2550 4450 0    50   ~ 0
+ESP_TX
+Wire Wire Line
+	2550 4450 3000 4450
+NoConn ~ 4650 2950
 $EndSCHEMATC
